Commit message: 20231113

File: omo_r1_description/urdf/omo_r1.urdf (robot description, URDF)
Before this commit: robot omo_r1, 11 links, 10 joints
Links:
- removed link camera_link
- removed link camera_rgb_frame
- removed link camera_rgb_optical_frame
Joints:
- removed joint camera_joint
- removed joint camera_rgb_joint
- removed joint camera_rgb_optical_joint
- joint base_joint: origin xyz=0 0.0 0.07 rpy=0 0 0.0 -> xyz=0 0 0.065 rpy=0 0 0
- joint wheel_left_joint: origin xyz=0.0 0.275 0.037 rpy=0.0 0.0 0 -> xyz=0.0 0.285 0.035 rpy=0 0 0; type continuous -> fixed
- joint wheel_right_joint: origin xyz=0.0 -0.275 0.037 rpy=0.0 0 0 -> xyz=0.0 -0.285 0.035 rpy=0 0 0; type continuous -> fixed

Commit message: 20231119

File: omo_r1_description/urdf/omo_r1.urdf (robot description, URDF)
Before this commit: robot omo_r1, 11 links, 10 joints
Links:
- removed link camera_link
- removed link camera_rgb_frame
- removed link camera_rgb_optical_frame
- link base_link: mass 8.2573504 -> None; geometry collision mesh filename=package://omo_r1_description/meshes/bases/omo_r2_body.stl scale=0.001 0.001 0.001; visual mesh filename=package://omo_r1_description/meshes/bases/omo_r2_body.stl scale=0.001 0.001 0.001
- link base_scan: mass 0.114 -> None; geometry 
- link caster_back_left_link: mass 0.000005 -> None
- link caster_back_right_link: mass 0.000005 -> None
- link wheel_left_link: mass 2.8498940 -> None; geometry collision mesh filename=package://omo_r1_description/meshes/wheels/omo_r2_wheel.stl scale=0.001 0.001 0.001; visual mesh filename=package://omo_r1_description/meshes/wheels/omo_r2_wheel.stl scale=0.001 0.001 0.001
- link wheel_right_link: mass 2.8498940 -> None; geometry collision mesh filename=package://omo_r1_description/meshes/wheels/omo_r2_wheel.stl scale=0.001 0.001 0.001; visual mesh filename=package://omo_r1_description/meshes/wheels/omo_r2_wheel.stl scale=0.001 0.001 0.001
Joints:
- removed joint camera_joint
- removed joint camera_rgb_joint
- removed joint camera_rgb_optical_joint
- joint base_joint: origin xyz=0 0.0 0.07 rpy=0 0 0.0 -> xyz=0.0 0.0 0.0635 rpy=0.0 0.0 0.0
- joint caster_back_left_joint: origin xyz=-0.33 0.148 0.06 rpy=0 0 0 -> xyz=-0.438 0.1347 -0.006 rpy=0 0 0
- joint caster_back_right_joint: origin xyz=-0.33 -0.148 0.06 rpy=0 0 0 -> xyz=-0.438 -0.1347 -0.006 rpy=0.0 0.0 0.0
- joint imu_joint: origin xyz=0.0 0 0.190 rpy=0 0 1.5758 -> xyz=-0.0065 0 0.128 rpy=0 0 1.5758
- joint scan_joint: origin xyz=0.06 0 0.230 rpy=0.0 0 3.14159 -> xyz=0.0 0.0 0.2585 rpy=0.0 0 3.14159
- joint wheel_left_joint: origin xyz=0.0 0.275 0.037 rpy=0.0 0.0 0 -> xyz=0.0 0.285 0.037 rpy=0.0 0.0 0.0
- joint wheel_right_joint: origin xyz=0.0 -0.275 0.037 rpy=0.0 0 0 -> xyz=0.0 -0.285 0.037 rpy=0.0 0.0 0.0
